Commit message: Add hook mesh

File: urdf/test_gripper.urdf (robot description, URDF)
Before this commit: robot test_gripper, 2 links, 1 joints
Links:
- link gripper: geometry collision mesh filename=package://hook_gripper_gazebo/meshes/hook_gripper.dae; visual mesh filename=package://hook_gripper_gazebo/meshes/hook_gripper.dae
Joints:
- joint joint: origin xyz=0 0 0 rpy=0 0 0 -> xyz=0 0 0 rpy=3.14 0 0
