Commit message: Add an example how to add gripper to a robot

File: robots/gripper.urdf.xacro (robot description, xacro)
@@ -1,14 +1,17 @@
 <?xml version="1.0"?>
-<robot name="test_gripper" xmlns:xacro="http://www.ros.org/wiki/xacro">
+<robot name="hook_gripper" xmlns:xacro="http://www.ros.org/wiki/xacro">
+  <xacro:include filename="$(find hook_gripper_gazebo)/urdf/hook_gripper.urdf.xacro" />
+  <xacro:arg name="prefix" default="" />
+  <!-- Desribe 1-dof robot -->
   <link name="world" />
   <joint name="joint" type="prismatic">
     <origin xyz="0 0 0" rpy="3.14 0 0" />
     <parent link="world" />
-    <child link="gripper" />
+    <child link="tool0" />
     <axis xyz="0 0 1" />
     <limit effort="300" velocity="1.0" lower="-1" upper="1" />
     <dynamics damping="0.0" />
   </joint>
-  <link name="gripper">
+  <link name="tool0">
     <inertial>
       <origin xyz="0 0 0" rpy="0 0 0" />
@@ -19,9 +22,8 @@
       <origin xyz="0 0 0" rpy="0 0 0" />
       <geometry>
-        <!-- <cylinder radius="0.05" length="0.1" /> -->
-        <mesh filename="package://hook_gripper_gazebo/meshes/hook_gripper.dae"/>
+        <cylinder radius="0.05" length="0.01" />
       </geometry>
       <material name="Grey">
-        <color rgba="0.3 0.3 0.3 1.0" />
+        <color rgba="1.0 0.3 0.3 1.0" />
       </material>
     </visual>
@@ -29,6 +31,5 @@
       <origin xyz="0 0 0" rpy="0 0 0" />
       <geometry>
-        <!-- <cylinder radius="0.05" length="0.1" /> -->
-        <mesh filename="package://hook_gripper_gazebo/meshes/hook_gripper.dae"/>
+        <cylinder radius="0.05" length="0.01" />
       </geometry>
     </collision>
@@ -43,20 +44,4 @@
     </actuator>
   </transmission>
-  <gazebo reference="gripper">
-    <material>Gazebo/Green</material>
-    <mu1>0.0</mu1>
-    <mu2>0.0</mu2>
-    <kp>0</kp>
-    <kd>0</kd>
-  </gazebo>
-  <gazebo>
-    <plugin name="hook_gripper" filename="libhook_gripper_gazebo.so">
-      <gripper_robot_name>test_gripper</gripper_robot_name>
-      <gripper_link_name>gripper</gripper_link_name>
-      <objects_robot_name>box</objects_robot_name>
-      <objects_link_name>box1</objects_link_name>
-      <min_collision_depth>0.001</min_collision_depth>
-    </plugin>
-  </gazebo>
   <gazebo>
     <plugin name="ros_control" filename="libgazebo_ros_control.so">
@@ -64,3 +49,5 @@
     </plugin>
   </gazebo>
+  <!-- connect to 1-dof robot The Hook fripper -->
+  <xacro:hook_gripper prefix="$(arg prefix)" parent="tool0" obj="box" obj_link="box1" />
 </robot>

Commit message: Add xacro insert origin to connect gripper to robot

File: robots/gripper.urdf.xacro (robot description, xacro)
@@ -49,5 +49,7 @@
     </plugin>
   </gazebo>
-  <!-- connect to 1-dof robot The Hook fripper -->
-  <xacro:hook_gripper prefix="$(arg prefix)" parent="tool0" obj="box" obj_link="box1" />
+  <!-- connect to 1-dof robot The Hook gripper -->
+  <xacro:hook_gripper prefix="$(arg prefix)" parent="tool0" obj="box" obj_link="box1">
+    <origin xyz="0 0 0" rpy="0 0 0"/>
+  </xacro:hook_gripper>
 </robot>

File: urdf/hook_gripper.urdf.xacro (robot description, xacro)
@@ -2,9 +2,10 @@
 <robot name="hook_gripper" xmlns:xacro="http://www.ros.org/wiki/xacro">
   <xacro:property name="M_PI" value="3.1415926535897931" />
-  <xacro:macro name="hook_gripper" params="prefix parent obj:=box obj_link:=box1">
+  <xacro:macro name="hook_gripper" params="prefix parent *origin obj:=box obj_link:=box1">
     <joint name="${prefix}joint_to_arm" type="revolute">
-      <origin xyz="0 0 0" rpy="0 0 0" />
+      <!-- <origin xyz="0 0 0" rpy="0 0 0" /> -->
+      <xacro:insert_block name="origin"/>
       <parent link="${parent}" />
-      <child link="gripper" />
+      <child link="${prefix}gripper" />
       <axis xyz="0 0 1" />
       <limit effort="1" velocity="1.0" lower="0" upper="0" />
@@ -21,5 +22,5 @@
         <geometry>
           <!-- <cylinder radius="0.05" length="0.1" /> -->
-          <mesh filename="package://hook_gripper_gazebo/meshes/hook_gripper.dae" />
+          <mesh filename="package://hook_gripper_gazebo/meshes/hook_gripper.dae" scale="1.05 1.05 1.05"/>
         </geometry>
         <material name="Grey">
@@ -31,10 +32,10 @@
         <geometry>
           <!-- <cylinder radius="0.05" length="0.1" /> -->
-          <mesh filename="package://hook_gripper_gazebo/meshes/hook_gripper.dae" />
+          <mesh filename="package://hook_gripper_gazebo/meshes/hook_gripper.dae" scale="1.05 1.05 1.05"/>
         </geometry>
       </collision>
     </link>
     <gazebo reference="${prefix}gripper">
-      <material>Gazebo/Green</material>
+      <material>Gazebo/Grey</material>
       <mu1>0.0</mu1>
       <mu2>0.0</mu2>
